File: PCB/klor1_3_kyle.kicad_pro/klor1_3_kyle.kicad_pro.kicad_sch (KiCad schematic)
At the start: 80 parts, among them J1 MJ-4PP-9, J3 lv27, SW1 SW_PUSH-MX_W_LED, SW10 SW_PUSH-MX_W_LED, SW11 SW_PUSH-MX_W_LED, SW12 SW_PUSH-MX_W_LED, SW13 SW_PUSH-MX_W_LED, SW14 SW_PUSH-MX_W_LED, SW15 SW_PUSH-MX_W_LED, SW16 SW_PUSH-MX_W_LED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

Commit message: Almost done!
Parts:
- added D23: D_Small, kbd:1N4148_SMD_both_side, symbol Device:D_Small
- added JP10, JP11: Device_Jumper_NO_Small, KLOR:Jumper, symbol KLORlib:Device_Jumper_NO_Small
- added SW23: SW_PUSH-MX_W_LED, keyswitches.pretty-master:1U_cherry_mx_kailh_choc_hotswap_combo, symbol KLORlib:SW_PUSH-MX_W_LED
Connections:
- net ENCB: now also JP11.1; no longer SW18.B
- net GND: now also JP10.1; no longer SW18.C
- net col0: now also SW23.5
- net col1: now also D23.1 (K)
- new net: D23.2 (A), SW23.6
- new net ENC_L: JP10.2, SW18.C
- new net ENC_R: JP11.2, SW18.B
Other:
- moved on the sheet: SW18
